File: main.sch (EAGLE design)
At the start: 14 parts, among them IC1 TS520550, IC2 TINY13-20SSU, J1 AVR_SPI_PROG_5X2PTH, T1 BST82-1

Commit message: Larger MOSFET, smaller SPI header and a rearrange.
Parts:
- removed U$1: A1SHB, Test:A1SHB
- removed VR1: 10k, SparkFun-Resistors:TRIMPOT-PTH-10MM-KNOB-1/2W-10%
- added C5: 0.1uF, SparkFun-Capacitors:0.1UF-0603-25V-5%
- added J5: AVR_SPI_PROG_3X2NS, SparkFun-Connectors:AVR_SPI_PROG_3X2NS
- added Q1: IRF4905, transistor-power:IRF4905
- added R2: 1k, SparkFun-Resistors:1KOHM-0603-1/10W-1%
- added S1: MOMENTARY-SWITCH-SPST-SMD-6.0X3.5MM, SparkFun-Switches:MOMENTARY-SWITCH-SPST-SMD-6.0X3.5MM
- J1: value AVR_SPI_PROG_5X2PTH -> (none); device SparkFun-Connectors:AVR_SPI_PROG_5X2PTH -> SparkFun-Connectors:CONN_03
Connections:
- net +5V: now also J1.3, R2.2; no longer VR1.CCW
- net 5VREG: now also C5.1
- net 5VSPI: now also J5.2; no longer J1.VCC
- net CLK: now also J5.3; no longer J1.SCK
- net GND: now also J1.1, J5.6, S1.1; no longer J1.GND@1, J1.GND@2, J1.GND@3, J1.GND@4, VR1.CW
- net MISO: now also J5.4; no longer J1.MISO
- net MOSI: now also J5.1; no longer J1.MOSI
- net N$1: now also Q1.D; no longer U$1.D
- net N$2: now also J1.2; no longer VR1.WIPER
- net N$3: now also Q1.G; no longer U$1.G
- net RESET: now also J5.5, R2.1, S1.2; no longer J1.RESET
- net VCC: now also C5.2, Q1.S; no longer U$1.S
